File: output/pcbs/left.kicad_pcb (KiCad board)
At the start: 2 copper layers, 159.8 x 104 mm, 80 parts

Commit message: adding tenting puck
Parts:
- removed ? (x5): , HOLE_M2_TH
- moved D29 12.4 mm to (220.3, 109.8)
- moved D30 6.19 mm to (220.3, 121.0)
- moved OLED1 0.79 mm to (239.5, 102.0)
- moved B1 0.65 mm to (244.5, 111.8)
Routing:
- net P111: track 388.6 -> 0.00 mm
- net P022: track 320.4 -> 0.00 mm
- net P020: track 308.7 -> 0.00 mm
- net P024: track 300.4 -> 0.00 mm
- net P113: track 204.6 -> 0.00 mm
- net P115: track 193.8 -> 0.00 mm
- net P031: track 185.3 -> 0.00 mm
- net P100: track 179.1 -> 0.00 mm
- net P002: track 176.8 -> 0.00 mm
- net P017: track 175.1 -> 0.00 mm
- net P011: track 162.4 -> 0.00 mm
- net P029: track 160.6 -> 0.00 mm
- net GND: track 98.0 -> 0.00 mm
- net RAW: track 79.0 -> 0.00 mm, vias 3 -> 0
- net RST: track 38.7 -> 0.00 mm
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Other:
- net class Default added: clearance 0.2, trace_width 0.25, via_dia 0.8, via_drill 0.4
